Commit message: fix: correct CI-05 J6 axis and dual-arm stand configuration

File: ros2_ws/src/iimt_dual_description/urdf/ci05_arm.xacro (robot description, xacro)
@@ -196,5 +196,5 @@
     <parent link="${prefix}wrist_2_link" />
     <child link="${prefix}wrist_3_link" />
-    <axis xyz="0 0 -1" />
+    <axis xyz="0 0 1" />
     <limit lower="-6.2832" upper="6.2832" effort="35" velocity="3.14" />
   </joint>

File: ros2_ws/src/iimt_ros2_description/urdf/iimt5.urdf (robot description, URDF)
Before this commit: robot iimt5, 7 links, 6 joints
Joints:
- joint wrist_3_joint: axis 0 0 -1 -> 0 0 1
